File: KiCAD/ardHotPlate/ardHotPlate.kicad_pcb (KiCad board)
At the start: 2 copper layers, 28 parts, among them T1 Transformer_dual_secondary_ce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, U1 LM348, U2 L7805, U3 L7905

Commit message: faulty diode footprint
Parts:
- D1: value ABS2 -> D_Bridge_+A-A
- moved D1 5.08 mm to (51.4, 31.8), turned to 270 degrees
Connections:
- D1 pad 2: Net-(C2-Pad2) -> Net-(D1-Pad2)
- D1 pad 3: Net-(D1-Pad3) -> Net-(C2-Pad2)
- F1 pad 1: Net-(D1-Pad4) -> Net-(D1-Pad2)
- F2 pad 1: Net-(D1-Pad3) -> Net-(D1-Pad4)
Routing:
- net Net-(C1-Pad1): track 62.7 -> 48.8 mm
- net Net-(D1-Pad2): track 0.00 -> 13.3 mm
- net Net-(D1-Pad3): track 11.7 -> 0.00 mm
- net Net-(C2-Pad2): track 66.2 -> 66.8 mm

Commit message: schematics
Other:
- net class Default removed
